Commit message: v1.0

File: hands/humanhand/humanhand.urdf (robot description, URDF)
Before this commit: robot human_hand, 26 links, 25 joints
Joints:
- joint index_joint1: limit lower=0 upper=1.57 effort=1 velocity=1 -> lower=-0.174532 upper=0.174532 effort=1 velocity=1
- joint index_joint2: limit lower=0 upper=1.57 effort=1 velocity=1 -> lower=-1.57 upper=1.57 effort=1 velocity=1
- joint middle_joint1: limit lower=0 upper=1.57 effort=1 velocity=1 -> lower=-0.174532 upper=0.174532 effort=1 velocity=1
- joint middle_joint2: limit lower=0 upper=1.57 effort=1 velocity=1 -> lower=-1.57 upper=1.57 effort=1 velocity=1
- joint pinky_joint1: limit lower=0 upper=1.57 effort=1 velocity=1 -> lower=-0.174532 upper=0.174532 effort=1 velocity=1
- joint pinky_joint2: limit lower=0 upper=1.57 effort=1 velocity=1 -> lower=-1.57 upper=1.57 effort=1 velocity=1
- joint ring_joint2: limit lower=0 upper=1.57 effort=1 velocity=1 -> lower=-1.57 upper=1.57 effort=1 velocity=1
- joint thumb_joint1: limit lower=0 upper=1.57 effort=1 velocity=1 -> lower=-0.174532 upper=0.174532 effort=1 velocity=1
- joint thumb_joint2: limit lower=0 upper=1.57 effort=1 velocity=1 -> lower=-1.57 upper=1.57 effort=1 velocity=1
